File: lets_split/lets_split.sch (KiCad schematic (older format))
At the start: 60 parts, among them J1 3PIN, J2 6PIN, J3 3PIN, SW1 SW_PUSH, SW10 SW_PUSH, SW11 SW_PUSH, SW12 SW_PUSH, SW13 SW_PUSH, SW14 SW_PUSH, SW15 SW_PUSH, SW16 SW_PUSH, SW17 SW_PUSH, SW18 SW_PUSH, SW19 SW_PUSH, SW2 SW_PUSH, SW20 SW_PUSH, SW21 SW_PUSH, SW22 SW_PUSH, SW23 SW_PUSH, SW24 SW_PUSH, SW3 SW_PUSH, SW4 SW_PUSH, SW5 SW_PUSH, SW6 SW_PUSH, SW7 SW_PUSH, SW8 SW_PUSH, SW9 SW_PUSH, U1 TEENSY2.0, U2 HOLE, U3 HOLE, U4 HOLE, U5 HOLE

Commit message: Change controller ProMicro to MCP23017
Parts:
- removed J1, J3: 3PIN, prettylib:jumper, symbol 3PIN
- removed J2: 6PIN, footprint:4pin35mmAudio, symbol 6PIN
- removed U1: TEENSY2.0, footprint:TEENSY_2.0, symbol TEENSY2.0
- removed W1: TEST, prettylib:JUMPER_SMD_2DUB, symbol TEST
- removed W2: TEST_1P, Wire_Pads:SolderWirePad_single_2mmDrill, symbol TEST_1P
- added C1: 0.1u, Capacitors_SMD:C_0603, symbol C
- added J3: Conn_01x04, Pin_Headers:Pin_Header_Straight_1x04_Pitch2.54mm, symbol Conn_01x04
- added JP1, JP2, JP3, JP4, JP5, JP6: Jumper_NO_Small, Jumper:SolderJumper-2_P1.3mm_Open_Pad1.0x1.5mm, symbol Jumper_NO_Small
- added R3: 10k, Resistors_SMD:R_0603, symbol R
- added U1: MCP23017, Housings_DFN_QFN:QFN-28-1EP_6x6mm_Pitch0.65mm, symbol MCP23017
- D1, D10, D11, D12, D13, D14, D15, D16, D17, D18, D19, D2, D20, D21, D22, D23, D24, D3, D4, D5, D6, D7, D8, D9: footprint Diodes_ThroughHole:Diode_DO-41_SOD81_Horizontal_RM10 -> Diodes_SMD:D_SOD-123
- R1, R2: value R -> 10k; footprint footprint:RESISTOR -> Resistors_SMD:R_0603
Connections:
- net labels removed: data, xtradata
- wire segments 24 -> 69
